Commit message: Updated mesh paths in URDF and MJCF; added launch, RViz config, CMakeLists.txt, and package.xml

File: robot_models/kbot-v2/kbot-v2_descritption/urdf/robot.urdf (robot description, URDF)
Before this commit: robot kbotv2p0_nohands, 23 links, 22 joints
Links:
- link KB_C_501X_Left_Bayonet_Adapter_Hard_Stop: geometry collision mesh filename=package://kbot-v2_descritption/meshes/KB_C_501X_Left_Bayone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; visual mesh filename=package://kbot-v2_descritption/meshes/KB_C_501X_Left_Bayone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
- link KB_C_501X_Right_Bayonet_Adapter_Hard_Stop: geometry collision mesh filename=package://kbot-v2_descritption/meshes/KB_C_501X_Right_Bayon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; visual mesh filename=package://kbot-v2_descritption/meshes/KB_C_501X_Right_Bayon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
- link KB_D_501L_L_LEG_FOOT: geometry collision mesh filename=package://kbot-v2_descritption/meshes/KB_D_501L_L_LEG_FOOT.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; visual mesh filename=package://kbot-v2_descritption/meshes/KB_D_501L_L_LEG_FOOT.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
- link KB_D_501R_R_LEG_FOOT: geometry collision mesh filename=package://kbot-v2_descritption/meshes/KB_D_501R_R_LEG_FOOT.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; visual mesh filename=package://kbot-v2_descritption/meshes/KB_D_501R_R_LEG_FOOT.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
- link KC_C_104L_PitchHardstopDriven: geometry collision mesh filename=package://kbot-v2_descritption/meshes/KC_C_104L_PitchHardst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; visual mesh filename=package://kbot-v2_descritption/meshes/KC_C_104L_PitchHardst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
- link KC_C_104R_PitchHardstopDriven: geometry collision mesh filename=package://kbot-v2_descritption/meshes/KC_C_104R_PitchHardst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; visual mesh filename=package://kbot-v2_descritption/meshes/KC_C_104R_PitchHardst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
- link KC_C_202L: geometry collision mesh filename=package://kbot-v2_descritption/meshes/KC_C_202L.collision.s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; visual mesh filename=package://kbot-v2_descritption/meshes/KC_C_202L.stl
- link KC_C_202R: geometry collision mesh filename=package://kbot-v2_descritption/meshes/KC_C_202R.collision.s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; visual mesh filename=package://kbot-v2_descritption/meshes/KC_C_202R.stl
- link KC_C_401L_L_UpForearmDrive: geometry collision mesh filename=package://kbot-v2_descritption/meshes/KC_C_401L_L_UpForearm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; visual mesh filename=package://kbot-v2_descritption/meshes/KC_C_401L_L_UpForearm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
- link KC_C_401R_R_UpForearmDrive: geometry collision mesh filename=package://kbot-v2_descritption/meshes/KC_C_401R_R_UpForearm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; visual mesh filename=package://kbot-v2_descritption/meshes/KC_C_401R_R_UpForearm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
- link KC_D_102L_L_Hip_Yoke_Drive: geometry collision mesh filename=package://kbot-v2_descritption/meshes/KC_D_102L_L_Hip_Yoke_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; visual mesh filename=package://kbot-v2_descritption/meshes/KC_D_102L_L_Hip_Yoke_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
- link KC_D_102R_R_Hip_Yoke_Drive: geometry collision mesh filename=package://kbot-v2_descritption/meshes/KC_D_102R_R_Hip_Yoke_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; visual mesh filename=package://kbot-v2_descritption/meshes/KC_D_102R_R_Hip_Yoke_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
- link KC_D_301L_L_Femur_Lower_Drive: geometry collision mesh filename=package://kbot-v2_descritption/meshes/KC_D_301L_L_Femur_Low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; visual mesh filename=package://kbot-v2_descritption/meshes/KC_D_301L_L_Femur_Low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
- link KC_D_301R_R_Femur_Lower_Drive: geometry collision mesh filename=package://kbot-v2_descritption/meshes/KC_D_301R_R_Femur_Low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; visual mesh filename=package://kbot-v2_descritption/meshes/KC_D_301R_R_Femur_Low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
- link KC_D_401L_L_Shin_Drive: geometry collision mesh filename=package://kbot-v2_descritption/meshes/KC_D_401L_L_Shin_Driv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; visual mesh filename=package://kbot-v2_descritption/meshes/KC_D_401L_L_Shin_Driv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
- link KC_D_401R_R_Shin_Drive: geometry collision mesh filename=package://kbot-v2_descritption/meshes/KC_D_401R_R_Shin_Driv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; visual mesh filename=package://kbot-v2_descritption/meshes/KC_D_401R_R_Shin_Driv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
- link RS03_3: geometry collision mesh filename=package://kbot-v2_descritption/meshes/RS03_3.collision.stl; visual mesh filename=package://kbot-v2_descritption/meshes/RS03_3.stl
- link RS03_4: geometry collision mesh filename=package://kbot-v2_descritption/meshes/RS03_4.collision.stl; visual mesh filename=package://kbot-v2_descritption/meshes/RS03_4.stl
- link RS03_5: geometry collision mesh filename=package://kbot-v2_descritption/meshes/RS03_5.collision.stl; visual mesh filename=package://kbot-v2_descritption/meshes/RS03_5.stl
- link RS03_6: geometry collision mesh filename=package://kbot-v2_descritption/meshes/RS03_6.collision.stl; visual mesh filename=package://kbot-v2_descritption/meshes/RS03_6.stl
- link Torso_Side_Right: geometry collision mesh filename=package://kbot-v2_descritption/meshes/Torso_Side_Right.coll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; visual mesh filename=package://kbot-v2_descritption/meshes/Torso_Side_Right.stl
- link imu: geometry collision mesh filename=package://kbot-v2_descritption/meshes/imu.collision.stl; visual mesh filename=package://kbot-v2_descritption/meshes/imu.stl
